File: kicad/phalwol.kicad_pcb (KiCad board)
At the start: 2 copper layers, 169.6 x 116.9 mm, 114 parts, among them J1 AudioJack4, SW1 SW_Push, SW10 SW_Push, SW11 SW_Push, SW12 SW_Push, SW13 SW_Push, SW14 SW_Push, SW15 SW_Push, SW16 SW_Push, SW17 SW_Push, SW18 SW_Push, SW19 SW_Push, SW2 SW_Push, SW20 SW_Push, SW21 SW_Push, SW22 SW_Push, SW23 SW_Push, SW24 SW_Push, SW25 SW_Push, SW26 SW_Push, SW27 SW_Push, SW28 SW_Push, SW29 SW_Push, SW3 SW_Push, SW30 SW_Push, SW31 SW_Push, SW32 SW_Push, SW33 SW_Push, SW34 SW_Push, SW35 SW_Push, SW36 SW_Push, SW37 SW_Push, SW38 SW_Push, SW39 SW_Push, SW4 SW_Push, SW40 SW_Push, SW41 SW_Push, SW5 SW_Push, SW6 SW_Push, SW7 SW_Push, SW8 SW_Push, SW9 SW_Push, U1 ProMicro

Commit message: hotfix wiring
Parts:
- removed the REF** at (80.1, 87.5)
- added REF**: MX_1u, yubuGadgetsFootpints:MX_1u, F.Cu at (54.0, 87.5)
- added REF**: Val**, yubuGadgetsFootpints:MX_HotswapOneside_Via_Guided, B.Cu at (75.4, 87.5)
- turned SW18 to 0 degrees
Routing:
- net Net-(D18-A): track 35.6 -> 29.0 mm
- net ROW4: track 241.5 -> 246.6 mm, vias 3 -> 5
- net ROW3: track 165.3 -> 170.3 mm, vias 2 -> 4
- net COL7: track 296.0 -> 300.6 mm
- net COL6: track 222.8 -> 227.1 mm
- net RST: track 120.2 -> 123.7 mm
- net COL2: track 188.4 -> 187.8 mm
- net GND: vias 52 -> 57
